File: popstar-rp2040/popstar.kicad_sch (KiCad schematic)
At the start: 31 parts, among them J1 JST SH 4-pin, J2 SWD, SW1 Boot, U2 XC6206PxxxMR, U3 SRV05-4, U4 W25Q128JVS, U6 RP2040, Y1 12MHz

Commit message: Added LCSC part for LEDs, gerber files for prod
Parts:
- U6: LCSC (none) -> C2040
Changed lines of the file:
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@@
       (effects (font (size 1.27 1.27)) (justify left bottom) hide)
+    )
+    (property "LCSC" "C2040" (at 64.77 83.82 0)
+      (effects (font (size 1.27 1.27)) hide)
     )
     (pin "1")
